Commit message: Update

File: urdf/g1_29dof_no_hands.urdf (robot description, URDF)
Before this commit: robot g1_29dof, 38 links, 37 joints
Links:
- added link left_tool_attach
- added link left_tool_connector_link, mass 0.01; collision cylinder length=0.022 radius=0.041; visual cylinder length=0.022 radius=0.041
- added link right_tool_attach
- added link right_tool_connector_link, mass 0.01; collision cylinder length=0.022 radius=0.041; visual cylinder length=0.022 radius=0.041
Joints:
- added joint left_tool_attach_joint: type fixed, parent left_tool_connector_link, child left_tool_attach, origin xyz=0.022 0 0 rpy=0 0 0
- added joint left_tool_connector_joint: type fixed, parent left_wrist_yaw_link, child left_tool_connector_link, origin xyz=0.0415 0.003 0 rpy=0 0 0
- added joint right_tool_attach_joint: type fixed, parent right_tool_connector_link, child right_tool_attach, origin xyz=0.022 0 0 rpy=0 0 0
- added joint right_tool_connector_joint: type fixed, parent right_wrist_yaw_link, child right_tool_connector_link, origin xyz=0.0415 -0.003 0 rpy=0 0 0

Commit message: Update

File: urdf/g1_29dof_no_hands.urdf (robot description, URDF)
Before this commit: robot g1_29dof, 42 links, 41 joints
Joints:
- joint left_tool_connector_joint: origin xyz=0.0415 0.003 0 rpy=0 0 0 -> xyz=0.0415 0.003 0 rpy=0 1.570796327 0
- joint right_tool_connector_joint: origin xyz=0.0415 -0.003 0 rpy=0 0 0 -> xyz=0.0415 -0.003 0 rpy=0 1.570796327 0

Commit message: Update

File: urdf/g1_29dof_no_hands.urdf (robot description, URDF)
Before this commit: robot g1_29dof, 42 links, 41 joints
Joints:
- joint left_tool_connector_joint: origin xyz=0.0415 0.003 0 rpy=0 1.570796327 0 -> xyz=0.0415 0.003 0 rpy=0 0 0
- joint right_tool_connector_joint: origin xyz=0.0415 -0.003 0 rpy=0 1.570796327 0 -> xyz=0.0415 -0.003 0 rpy=0 0 0

Commit message: Update

File: urdf/g1_29dof_no_hands.urdf (robot description, URDF)
Before this commit: robot g1_29dof, 42 links, 41 joints
Links:
- link left_tool_connector_link: geometry collision mesh filename=package://g1_description/meshes/tool_connector_cyl_x.STL; visual mesh filename=package://g1_description/meshes/tool_connector_cyl_x.STL
- link right_tool_connector_link: geometry collision mesh filename=package://g1_description/meshes/tool_connector_cyl_x.STL; visual mesh filename=package://g1_description/meshes/tool_connector_cyl_x.STL

Commit message: Update

File: urdf/g1_29dof_no_hands.urdf (robot description, URDF)
Before this commit: robot g1_29dof, 42 links, 41 joints
Joints:
- joint left_tool_attach_joint: origin xyz=0.022 0 0 rpy=-1.5707963267948966 1.5707963267948966 0 -> xyz=0.022 0 0 rpy=0 1.5707963267948966 0
- joint right_tool_attach_joint: origin xyz=0.022 0 0 rpy=1.5707963267948966 1.5707963267948966 0 -> xyz=0.022 0 0 rpy=0 1.5707963267948966 0

Commit message: Update

File: urdf/g1_29dof_no_hands.urdf (robot description, URDF)
Before this commit: robot g1_29dof, 42 links, 41 joints
Joints:
- joint left_tool_attach_joint: origin xyz=0.022 0 0 rpy=0 1.5707963267948966 0 -> xyz=0.022 0 0 rpy=-1.5707963267948966 0 -1.5707963267948966
- joint right_tool_attach_joint: origin xyz=0.022 0 0 rpy=0 1.5707963267948966 0 -> xyz=0.022 0 0 rpy=1.5707963267948966 0 1.5707963267948966
